File: LEDSubMatrixHighDensity/LEDSubMatrixHighDensity_scripttesting.sch (EAGLE design)
At the start: 129 parts, among them IC1 TLC5955DCAR, IC2 TLC5955DCAR, IC3 TLC5955DCAR, IC4 TLC5955DCAR, IC5 TLC5955DCAR, IC6 TLC5955DCAR, IC7 TLC5955DCAR, IC8 TLC5955DCAR

Commit message: Finished placing all LEDs and Led Drivers
Parts:
- SV1: device con-lstb:MA04-2 -> con-lstb:MA06-2
Connections:
- removed net SIN_MCU: IC1.SIN, IC2.SIN, IC3.SIN, IC4.SIN, IC5.SIN, IC6.SIN, IC7.SIN, IC8.SIN, SV1.8
- new net N$9: SV1.5
- new net SIN_1,2: IC1.SIN, IC2.SIN
- new net SIN_3,4: IC3.SIN, IC4.SIN
- new net SIN_5,6: IC5.SIN, IC6.SIN
- new net SIN_7,8: IC7.SIN, IC8.SIN
- new net SOUT2: IC2.SOUT
- new net SOUT3: IC3.SOUT
- new net SOUT4: IC4.SOUT
- new net SOUT5: IC5.SOUT
- new net SOUT6: IC6.SOUT
- new net SOUT7: IC7.SOUT
- new net SOUT8: IC8.SOUT
- net 3V3: now also SV1.10, SV1.9; no longer SV1.4
- net GND: now also SV1.11, SV1.12; no longer SV1.2
- net GSCLK: now also SV1.6; no longer SV1.5
- net LAT: now also SV1.4, SV1.8
- net SCLK: now also SV1.2, SV1.7; no longer SV1.6
- net SOUT1: no longer IC2.SOUT, IC3.SOUT, IC4.SOUT, IC5.SOUT, IC6.SOUT, IC7.SOUT, IC8.SOUT, SV1.7
Other:
- note added: "ADD DECOUPLING CAPACITORS at power bridge (10uF)"
- moved on the sheet: IC1, IC2, IC3, IC4, IC5, IC6, IC7, IC8, LED1, LED10, LED100, LED105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
