File: LEDSubMatrixHighDensity/LEDSubMatrixHighDensity_template.brd (EAGLE design)
At the start: 17 parts, among them IC1 TLC5955DCAR

Commit message: added pictures of led matrix pcbs
Routing:
- net 3V3: track 0.00 -> 3.66 mm, vias 0 -> 1
- net N$LEDB11_IC1_PIN41: track 0.00 -> 3.57 mm, vias 0 -> 1
- net SCLK: track 0.00 -> 1.74 mm, vias 0 -> 1
- net N$LEDG16_IC1_PIN30: track 6.28 -> 4.60 mm
- net N$LEDB16_IC1_PIN32: track 8.16 -> 6.60 mm
- net N$LEDR16_IC1_PIN31: track 5.66 -> 4.31 mm
- net N$LEDB12_IC1_PIN35: track 7.00 -> 5.72 mm
- net N$LEDB9_IC1_PIN53: track 2.35 -> 3.60 mm
- net SIN_MCU: track 0.00 -> 1.24 mm, vias 0 -> 1
- net LAT: track 0.00 -> 1.24 mm, vias 0 -> 1
- net N$LEDB8_IC1_PIN25: track 6.52 -> 5.39 mm
- net N$LEDB15_IC1_PIN38: track 7.03 -> 6.11 mm
- net N$LEDB14_IC1_PIN44: track 7.15 -> 6.24 mm
- net N$LEDB13_IC1_PIN50: track 7.30 -> 7.99 mm
- net N$LEDG12_IC1_PIN33: track 4.50 -> 3.82 mm
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- added copper zone on layer 16, net GND
Other:
- board outline added: 16.9 x 127 mm

Commit message: Finished placing all LEDs and Led Drivers
Routing:
- net N$LEDR5_IC1_PIN8: track 6.38 -> 9.85 mm
- net SCLK: track 1.74 -> 0.00 mm, vias 1 -> 0
- net SIN_MCU: track 1.24 -> 0.00 mm, vias 1 -> 0
- net LAT: track 1.24 -> 0.00 mm, vias 1 -> 0
- net N$LEDB12_IC1_PIN35: track 5.72 -> 6.65 mm
- net N$LEDG14_IC1_PIN42: track 5.52 -> 6.44 mm
- net N$LEDR6_IC1_PIN14: track 6.77 -> 7.57 mm
- net N$LEDB13_IC1_PIN50: track 7.99 -> 8.74 mm
- net 3V3: track 3.66 -> 3.01 mm
- net N$LEDR4_IC1_PIN23: track 2.43 -> 3.04 mm
- net N$LEDR12_IC1_PIN34: track 3.07 -> 3.65 mm
- net N$LEDG13_IC1_PIN48: track 5.87 -> 6.39 mm
