File: LEDSubMatrixLowDensitySMD/LEDSubMatrixLowDensitySMD.brd (EAGLE design)
At the start: 50.8 x 146 mm, 70 parts, among them IC1 TLC5955DCAR, IC2 TLC5955DCAR, IC3 TLC5955DCAR

Commit message: fixed problem of not having pairs of drivers daisy-chained
Parts:
- moved R9 63.3 mm to (12.0, -89.0), flipped to the top
- moved R14 57.8 mm to (13.5, -126.4), flipped to the top, turned to 270 degrees
- moved R10 54.5 mm to (28.0, -74.0), flipped to the top
- moved R6 53.7 mm to (17.0, -74.0), flipped to the top
- moved R16 53.0 mm to (38.0, -74.0), flipped to the top
- moved R8 53.0 mm to (22.0, -74.0), flipped to the top
- moved R7 48.4 mm to (33.0, -74.0), flipped to the top
- moved R11 39.1 mm to (17.0, -112.0), flipped to the top
- moved R13 38.1 mm to (22.0, -112.0), flipped to the top
- moved R17 38.1 mm to (38.0, -112.0), flipped to the top
- moved R15 36.1 mm to (28.0, -112.0), flipped to the top
- moved R12 35.2 mm to (33.0, -112.0), flipped to the top
- moved R4 22.0 mm to (13.3, -38.0), flipped to the top, turned to 270 degrees
- moved R2 10.7 mm to (33.5, -23.1), flipped to the top
- moved R18 3.98 mm to (38.5, -23.1), flipped to the top
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Connections:
- net N$LEDB41_IC3_PIN53 renamed N$1
- net N$LEDB42_IC3_PIN47 renamed N$16
- net N$LEDB43_IC3_PIN41 renamed N$22
- net N$LEDB44_IC3_PIN35 renamed N$28
- net N$LEDB45_IC3_PIN50 renamed N$9
- net N$LEDB46_IC3_PIN44 renamed N$19
- net N$LEDB47_IC3_PIN38 renamed N$25
- net N$LEDB48_IC3_PIN32 renamed N$31
- net N$LEDG41_IC3_PIN51 renamed N$6
- net N$LEDG42_IC3_PIN45 renamed N$18
- net N$LEDG43_IC3_PIN39 renamed N$24
- net N$LEDG44_IC3_PIN33 renamed N$30
- net N$LEDG45_IC3_PIN48 renamed N$14
- net N$LEDG46_IC3_PIN42 renamed N$21
- net N$LEDG47_IC3_PIN36 renamed N$27
- net N$LEDG48_IC3_PIN30 renamed N$33
- net N$LEDR41_IC3_PIN52 renamed N$4
- net N$LEDR42_IC3_PIN46 renamed N$17
- net N$LEDR43_IC3_PIN40 renamed N$23
- net N$LEDR44_IC3_PIN34 renamed N$29
- net N$LEDR45_IC3_PIN49 renamed N$11
- net N$LEDR46_IC3_PIN43 renamed N$20
- net N$LEDR47_IC3_PIN37 renamed N$26
- net N$LEDR48_IC3_PIN31 renamed N$32
Routing:
- net SOUT1: track 0.00 -> 152.8 mm, vias 0 -> 1
- net SOUT2: track 0.00 -> 99.3 mm, vias 0 -> 1
- net SOUT3: track 0.00 -> 71.5 mm, vias 0 -> 1
- net N$LEDB29_IC2_PIN50: track 0.00 -> 40.9 mm, vias 0 -> 1
- net N$LEDR13_IC1_PIN49: track 0.00 -> 37.6 mm, vias 0 -> 1
- net N$LEDB40_IC3_PIN25: track 0.00 -> 37.3 mm, vias 0 -> 1
- net N$LEDR40_IC3_PIN26: track 0.00 -> 35.9 mm, vias 0 -> 1
- net N$LEDR17_IC2_PIN5: track 0.00 -> 34.9 mm, vias 0 -> 1
- net N$LEDB32_IC2_PIN32: track 0.00 -> 33.7 mm, vias 0 -> 1
- net N$LEDR1_IC1_PIN5: track 0.00 -> 33.1 mm, vias 0 -> 3
- net N$LEDG5_IC1_PIN9: track 0.00 -> 28.0 mm, vias 0 -> 1
- net N$LEDR20_IC2_PIN23: track 0.00 -> 27.9 mm, vias 0 -> 1
- net N$LEDG4_IC1_PIN24: track 0.00 -> 27.7 mm, vias 0 -> 1
- net N$LEDB4_IC1_PIN22: track 0.00 -> 27.2 mm, vias 0 -> 1
- net N$LEDG20_IC2_PIN24: track 0.00 -> 27.2 mm, vias 0 -> 1
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