File: LEDSubMatrix_rev2/LEDSubMatrixHighDensity/LEDSubMatrixHighDensity_test.sch (EAGLE design)
At the start: 145 parts, among them IC1 TLC5955DCAR, IC2 TLC5955DCAR, IC3 TLC5955DCAR, IC4 TLC5955DCAR, IC5 TLC5955DCAR, IC6 TLC5955DCAR, IC7 TLC5955DCAR, IC8 TLC5955DCAR

Commit message: finished rev 2 of PCB submatrix led
Connections:
- removed net 3V3_LOGIC: C1.1, C1B.1, C2.1, C2B.1, C3.1, C3B.1, C4.1, C4B.1, C5.1, C5B.1, C6.1, C6B.1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
- net 3V3: now also C1.1, C1B.1, C2.1, C2B.1, C3.1, C3B.1, C4.1, C4B.1, C5.1, C5B.1, C6.1, C6B.1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
- net GND: now also SV1.9
