File: LEDSubMatrix_rev2/LEDSubMatrixHighDensity/LEDSubMatrixHighDensity_v2.brd (EAGLE design)
At the start: 16.9 x 146 mm, 145 parts, among them IC1 TLC5955DCAR, IC2 TLC5955DCAR, IC3 TLC5955DCAR, IC4 TLC5955DCAR, IC5 TLC5955DCAR, IC6 TLC5955DCAR, IC7 TLC5955DCAR, IC8 TLC5955DCAR

Commit message: Added logic buffers to LED matrix
Parts:
- added C28, C30, C32: 0.1u, GTOR - Passive Components:C0603
- added C29, C31, C33: 4.7u, GTOR - Passive Components:C0603
- added IC10, IC11, IC9: SN74LVC1G34DBVR, SN74LVC1G34DBVR:SOT95P280X145-5N
Connections:
- new net GSCLK_FPGA: IC11.2, SV1.3
- new net LAT_FPGA: IC9.2, SV1.5
- new net SCLK_FPGA: IC10.2, SV1.7
- net 3V3_LOGIC: now also C28.1, C29.1, C30.1, C31.1, C32.1, C33.1, IC10.5, IC11.5, IC9.5
- net GND: now also C28.2, C29.2, C30.2, C31.2, C32.2, C33.2, IC10.3, IC11.3, IC9.3
- net GSCLK: now also IC11.4; no longer SV1.3
- net LAT: now also IC9.4; no longer SV1.5
- net SCLK: now also IC10.4; no longer SV1.7
Routing:
- net SCLK: track 155.8 -> 153.5 mm
