File: Controls/SpinningControls_4in_1_crammed.brd (EAGLE design)
At the start: 203.2 x 101.6 mm, 33 parts, among them IC1 S-19246E33H-V5T2U, IC2 SN74LVC1G34DBVR, IC3 SN74LVC1G34DBVR, IC4 SN74LVC1G34DBVR, J1 SULLINS_PPPC062LFBN-RCSULLINS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, J10 SULLINS_PPPC062LFBN-RCSULLINS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, J11 SULLINS_PPPC062LFBN-RCSULLINS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, J12 SULLINS_PPPC062LFBN-RCSULLINS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, J13 SULLINS_PPPC062LFBN-RCSULLINS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, J14 SULLINS_PPPC062LFBN-RCSULLINS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

Commit message: parts exchange, layout corrections, no routing
Parts:
- removed R4: 165 Ω, rcl:R0603
- removed U$4: DE0-NANO, VoxelEagleLib:DE0-NANO
- removed X2, X3: 5566-4, con-molex:5566-4
- removed X4: 5566-6, con-molex:5566-6
- added FPGA: DE0-NANO, VoxelEagleLib:DE0-NANO
- added J15: 430450612, molex:CON_430450612_MOL
- added J16, J17: 430450412, molex:CON_430450412_MOL
- added J18, J19: 436500215, molex:CON_436500215_MOL
- added R5: 19.1k Ω, rcl:R0402
- J1: value SULLINS_PPPC062LFBN-RCSULLINS_PPPC062LFBN-RC_0_0 -> 7-146256-0; device Sullins - PPPC062LFBN-RC:SULLINS_PPPC062LFBN-RC_0 -> SamacSys_Parts:HDRV40W67P254_2X20_5039X488X81
- J2: value 7-146256-0 -> F32R-1A7H1-11040; device SamacSys_Parts:HDRV40W67P254_2X20_5039X488X81 -> F32R-1A7H1-11040:F32R1A7H111040
- J3: value F32R-1A7H1-11040 -> SULLINS_PPPC062LFBN-RCSULLINS_PPPC062LFBN-RC_0_0; device F32R-1A7H1-11040:F32R1A7H111040 -> Sullins - PPPC062LFBN-RC:SULLINS_PPPC062LFBN-RC_0
- R3: value 165 Ω -> 19.1k Ω; device rcl:R0603 -> rcl:R0402
- moved R2 383.5 mm to (214.6, 68.6)
- moved R3 354.9 mm to (214.6, 73.7)
- moved R1 353.6 mm to (214.6, 83.8)
- moved IC4 336.3 mm to (194.3, 33.0)
- moved IC3 331.5 mm to (194.3, 38.1)
- moved IC2 326.8 mm to (194.3, 43.2)
- moved J3 280.0 mm to (191.8, 57.1), flipped to the bottom
- moved U$3 224.9 mm to (129.5, 72.4)
- moved J1 221.9 mm to (106.7, 50.8), turned to 270 degrees
- moved J9 219.8 mm to (92.7, 57.1), flipped to the bottom
- moved J8 218.6 mm to (109.2, 57.1), flipped to the bottom
- moved J7 217.5 mm to (125.7, 57.1), flipped to the bottom
- moved J6 216.3 mm to (142.2, 57.1), flipped to the bottom
- moved J5 215.1 mm to (158.8, 57.1), flipped to the bottom
- moved J4 214.0 mm to (175.3, 57.1), flipped to the bottom
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Connections:
- removed net N$25: R1.2, X2.1
- removed net N$26: R2.2, X3.1
- removed net N$27: R3.2, X2.3
- removed net N$28: R4.2, X3.3
- removed net N$30: X4.2
- new net N$1: J16.4, R5.1
- new net N$2: J17.4, R3.1
- new net N$5: J16.2, R1.1
- new net N$6: J17.2, R2.1
- net 24V: now also J15.2; no longer X4.5
- net 5V: now also J16.3, J17.3, J18.2, J19.2, R3.2, R5.2; no longer R1.1, R2.1, X2.2, X3.2
- net ACTIVE: now also J1.31
- net B1: now also J1.21
- net B2: now also J1.22
- net B3: now also J1.23
- net B4: now also J1.24
- net B5: now also J1.25
- net B6: now also J1.26
- net B7: now also J1.27
- net B8: now also J1.28
- net DISPEN: now also J1.34
- net ENC_POS: now also J15.4, R2.2; no longer R4.1
- net ENC_POS0: now also R1.2; no longer R3.1
- net G1: now also J1.13
- net G2: now also J1.14
- net G3: now also J1.15
- net G4: now also J1.16
- net G5: now also J1.17
- net G6: now also J1.18
- net G7: now also J1.19
- net G8: now also J1.20
- net GND: now also J15.1, J16.1, J17.1, J18.1, J19.1, U$1.6; no longer X2.4, X3.4, X4.6
- net HSYNC: now also J1.32
- net N$10: now also FPGA.30; no longer U$4.30
- net N$11: now also FPGA.51; no longer U$4.51
- net N$12: now also FPGA.69; no longer U$4.69
- net N$13: now also FPGA.52; no longer U$4.52
- net N$14: now also FPGA.70; no longer U$4.70
- net N$15: now also FPGA.98; no longer U$4.98
- net N$16: now also FPGA.100; no longer U$4.100
- net N$17: now also FPGA.102; no longer U$4.102
- net N$18: now also FPGA.104; no longer U$4.104
- net N$19: now also FPGA.99; no longer U$4.99
- net N$20: now also FPGA.101; no longer U$4.101
- net N$21: now also FPGA.103; no longer U$4.103
- net N$22: now also FPGA.105; no longer U$4.105
- net N$23: now also FPGA.81; no longer U$4.81
- net N$24: now also FPGA.106; no longer U$4.106
- net N$3: now also FPGA.11; no longer U$4.11
- net N$7: now also FPGA.12; no longer U$4.12
- net N$9: now also FPGA.29; no longer U$4.29
- net PIXCLK: now also J1.30
- net PI_RX: now also J15.5
- net PI_TX: now also J15.6; no longer X4.1
- net R1: now also J1.5
- net R2: now also J1.6
- net R3: now also J1.7
- net R4: now also J1.8
- net R5: now also J1.9
- net R6: now also J1.10
- net R7: now also J1.11
- net R8: now also J1.12
- net VSYNC: now also J1.33
Routing:
- net N$8: track 0.00 -> 268.5 mm
