File: Controls/SpinningControls_4in_2_flipped.brd (EAGLE design)
At the start: 203.2 x 101.6 mm, 34 parts, among them IC1 S-19246E33H-V5T2U, IC2 SN74LVC1G34DBVR, IC3 SN74LVC1G34DBVR, IC4 SN74LVC1G34DBVR, J1 7-146256-0, J10 SULLINS_PPPC062LFBN-RCSULLINS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, J11 SULLINS_PPPC062LFBN-RCSULLINS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, J12 SULLINS_PPPC062LFBN-RCSULLINS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, J13 SULLINS_PPPC062LFBN-RCSULLINS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, J14 SULLINS_PPPC062LFBN-RCSULLINS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

Commit message: parts exchange, layout corrections, no routing
Parts:
- removed R4: 165 Ω, rcl:R0603
- removed X1: 22-23-2021, con-molex:22-23-2021
- removed X2, X3: 5566-4, con-molex:5566-4
- removed X4: 5566-6, con-molex:5566-6
- added J15: 430450612, molex:CON_430450612_MOL
- added J16, J17: 430450412, molex:CON_430450412_MOL
- added J18, J19: 436500215, molex:CON_436500215_MOL
- added R5: 19.1k Ω, rcl:R0402
- R3: value 165 Ω -> 19.1k Ω; device rcl:R0603 -> rcl:R0402
- moved J3 319.8 mm to (188.0, -12.7), flipped to the bottom
- moved U$2 274.0 mm to (139.7, 1.27), turned to 90 degrees
- moved J9 251.7 mm to (88.9, -12.7), flipped to the bottom
- moved J8 250.7 mm to (105.4, -12.7), flipped to the bottom
- moved J7 249.7 mm to (121.9, -12.7), flipped to the bottom
- moved J6 248.7 mm to (138.4, -12.7), flipped to the bottom
- moved J5 247.7 mm to (154.9, -12.7), flipped to the bottom
- moved J4 246.7 mm to (171.4, -12.7), flipped to the bottom
- moved J2 245.4 mm to (161.3, 85.1)
- moved C2 239.4 mm to (118.5, 32.4), turned to 180 degrees
- moved C3 234.3 mm to (122.9, 39.1)
- moved C1 227.2 mm to (118.5, 34.9), turned to 180 degrees
- moved J1 211.8 mm to (139.7, 95.2)
- moved IC4 204.6 mm to (43.2, 68.6), turned to 180 degrees
- moved R2 201.4 mm to (-8.89, 81.3), turned to 180 degrees
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Connections:
- removed net N$25: R1.2, X2.1
- removed net N$26: R2.2, X3.1
- removed net N$27: R3.2, X2.3
- removed net N$28: R4.2, X3.3
- new net N$1: J16.4, R5.1
- new net N$2: J17.4, R3.1
- new net N$5: J16.2, R1.1
- new net N$6: J17.2, R2.1
- net 24V: now also J15.2; no longer X4.5
- net 5V: now also J16.3, J17.3, J18.2, J19.2, R3.2, R5.2; no longer R1.1, R2.1, X1.2, X2.2, X3.2
- net ENC_POS: now also J15.4, R2.2; no longer R4.1, X4.3
- net ENC_POS0: now also R1.2; no longer R3.1
- net GND: now also J15.1, J16.1, J17.1, J18.1, J19.1; no longer X1.1, X2.4, X3.4, X4.6
- net PI_RX: now also J15.5; no longer X4.2
- net PI_TX: now also J15.6; no longer X4.1
Routing:
- net N$8: track 0.00 -> 268.5 mm
