File: Controls/SpinningControls.brd (EAGLE design)
At the start: 209.6 x 107.9 mm, 46 parts, among them IC1 S-19246E33H-V5T2U, IC2 SN74LVC1G34DBVR, IC3 SN74LVC1G34DBVR, IC4 SN74LVC1G34DBVR, J10 SULLINS_PPPC062LFBN-RCSULLINS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, J11 SULLINS_PPPC062LFBN-RCSULLINS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, J12 SULLINS_PPPC062LFBN-RCSULLINS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, J13 SULLINS_PPPC062LFBN-RCSULLINS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, J14 SULLINS_PPPC062LFBN-RCSULLINS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, J15 430450612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

Commit message: Finished power routing and other minor changes
Parts:
- R3, R4: device rcl:R0402 -> rcl:R0603
- moved C15 112.8 mm to (10.5, 61.1), flipped to the bottom, turned to 90 degrees
- moved C14 100.9 mm to (27.6, 61.1), flipped to the bottom, turned to 90 degrees
- moved C13 89.0 mm to (44.6, 61.1), flipped to the bottom, turned to 90 degrees
- moved C12 77.1 mm to (61.6, 61.1), flipped to the bottom, turned to 90 degrees
- moved C11 65.2 mm to (78.6, 61.1), flipped to the bottom, turned to 90 degrees
- moved C10 53.2 mm to (95.8, 61.1), flipped to the bottom, turned to 90 degrees
- moved C9 41.5 mm to (112.6, 61.1), flipped to the bottom, turned to 90 degrees
- moved C8 29.7 mm to (129.7, 61.1), flipped to the bottom, turned to 90 degrees
- moved C7 18.2 mm to (146.7, 61.1), flipped to the bottom, turned to 90 degrees
- moved C4 14.3 mm to (191.9, 61.1), flipped to the bottom, turned to 90 degrees
- moved C5 9.26 mm to (180.8, 61.1), flipped to the bottom, turned to 90 degrees
- moved C6 8.03 mm to (163.8, 61.1), flipped to the bottom, turned to 90 degrees
Routing:
- net 3V3_LOGIC: track 0.00 -> 449.4 mm, vias 0 -> 12
- net 5V: track 0.00 -> 397.4 mm, vias 0 -> 6
- net ENC_POS: track 0.00 -> 264.7 mm, vias 0 -> 1
- net ENC_POS0: track 0.00 -> 136.9 mm
- net SIN12_J3: track 0.00 -> 116.4 mm
- net SIN56_J3: track 0.00 -> 112.1 mm
- net SIN34_J3: track 0.00 -> 109.6 mm
- net SIN78_J3: track 0.00 -> 108.1 mm
- net PI_TX: track 0.00 -> 96.6 mm, vias 0 -> 1
- net PI_RX: track 0.00 -> 91.6 mm, vias 0 -> 1
- net 24V: track 0.00 -> 73.8 mm
- net SIN12_J6: track 0.00 -> 41.0 mm
- net GND: track 0.00 -> 33.0 mm, vias 0 -> 51
- net SIN56_J7: track 0.00 -> 25.6 mm
- net SIN12_J7: track 0.00 -> 24.7 mm
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- added copper zone on layer 1, net 3V3_LED
- added copper zone on layer 1, net GND

Commit message: Finished controls board, added gerbers
Routing:
- net GSCLK: track 0.00 -> 347.2 mm, vias 0 -> 13
- net LAT: track 0.00 -> 331.3 mm, vias 0 -> 13
- net SCLK: track 0.00 -> 316.4 mm, vias 0 -> 10
- net SIN12_J4: track 16.7 -> 107.0 mm
- net SIN56_J4: track 15.6 -> 105.1 mm
- net SIN34_J4: track 15.9 -> 102.7 mm
- net SIN12_J5: track 18.5 -> 105.3 mm
- net SIN56_J5: track 17.0 -> 103.7 mm
- net SIN78_J4: track 15.2 -> 101.2 mm
- net SIN34_J5: track 18.3 -> 101.4 mm
- net SIN78_J5: track 17.2 -> 100.0 mm
- net SIN56_J6: track 21.8 -> 103.9 mm
- net SIN34_J6: track 21.6 -> 101.4 mm
- net SIN78_J6: track 22.6 -> 100.3 mm
- net SIN12_J6: track 41.0 -> 105.0 mm
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