File: Controls/SpinningControls.sch (EAGLE design)
At the start: 46 parts, among them IC1 S-19246E33H-V5T2U, IC2 SN74LVC1G34DBVR, IC3 SN74LVC1G34DBVR, IC4 SN74LVC1G34DBVR, J10 SULLINS_PPPC062LFBN-RCSULLINS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, J11 SULLINS_PPPC062LFBN-RCSULLINS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, J12 SULLINS_PPPC062LFBN-RCSULLINS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, J13 SULLINS_PPPC062LFBN-RCSULLINS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, J14 SULLINS_PPPC062LFBN-RCSULLINS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, J15 430450612, J16 430450612, J17 430450612, J18 436500215, J19 436500215, J2 F32R-1A7H1-11040, J3 SULLINS_PPPC062LFBN-RCSULLINS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, J4 SULLINS_PPPC062LFBN-RCSULLINS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, J5 SULLINS_PPPC062LFBN-RCSULLINS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, J6 SULLINS_PPPC062LFBN-RCSULLINS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, J7 SULLINS_PPPC062LFBN-RCSULLINS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, J8 SULLINS_PPPC062LFBN-RCSULLINS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, J9 SULLINS_PPPC062LFBN-RCSULLINS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

Commit message: full schematic, silkscreen cleanup
Connections:
- net ENC_POS: now also FPGA.GPIO_0_IN0
- net ENC_POS0: now also FPGA.GPIO_0_IN1
- net G1: now also FPGA.GPIO_017; no longer FPGA.GPIO_030
- net G2: now also FPGA.GPIO_015; no longer FPGA.GPIO_028
- net G3: now also FPGA.GPIO_013; no longer FPGA.GPIO_026
- net G4: now also FPGA.GPIO_011; no longer FPGA.GPIO_024
- net G5: now also FPGA.GPIO_09; no longer FPGA.GPIO_022
- net GSCLK_FPGA: now also FPGA.GPIO_032
- net LAT_FPGA: now also FPGA.GPIO_132
- net R8: now also FPGA.GPIO_019; no longer FPGA.GPIO_032
- net SCLK_FPGA: now also FPGA.GPIO_133
- net SIN12_J10: now also FPGA.GPIO_116
- net SIN12_J11: now also FPGA.GPIO_112
- net SIN12_J12: now also FPGA.GPIO_18
- net SIN12_J13: now also FPGA.GPIO_14
- net SIN12_J14: now also FPGA.GPIO_10
- net SIN12_J3: now also FPGA.GPIO_07
- net SIN12_J4: now also FPGA.GPIO_014
- net SIN12_J5: now also FPGA.GPIO_022
- net SIN12_J6: now also FPGA.GPIO_030
- net SIN12_J7: now also FPGA.GPIO_128
- net SIN12_J8: now also FPGA.GPIO_124
- net SIN12_J9: now also FPGA.GPIO_120
- net SIN34_J10: now also FPGA.GPIO_117
- net SIN34_J11: now also FPGA.GPIO_113
- net SIN34_J12: now also FPGA.GPIO_19
- net SIN34_J13: now also FPGA.GPIO_15
- net SIN34_J14: now also FPGA.GPIO_11
- net SIN34_J3: now also FPGA.GPIO_06
- net SIN34_J4: now also FPGA.GPIO_012
- net SIN34_J5: now also FPGA.GPIO_020
- net SIN34_J6: now also FPGA.GPIO_028
- net SIN34_J7: now also FPGA.GPIO_129
- net SIN34_J8: now also FPGA.GPIO_125
- net SIN34_J9: now also FPGA.GPIO_121
- net SIN56_J10: now also FPGA.GPIO_118
- net SIN56_J11: now also FPGA.GPIO_114
- net SIN56_J12: now also FPGA.GPIO_110
- net SIN56_J13: now also FPGA.GPIO_16
- net SIN56_J14: now also FPGA.GPIO_12
- net SIN56_J3: now also FPGA.GPIO_04
- net SIN56_J4: now also FPGA.GPIO_010
- net SIN56_J5: now also FPGA.GPIO_018
- net SIN56_J6: now also FPGA.GPIO_026
- net SIN56_J7: now also FPGA.GPIO_130
- net SIN56_J8: now also FPGA.GPIO_126
- net SIN56_J9: now also FPGA.GPIO_122
- net SIN78_J10: now also FPGA.GPIO_119
- net SIN78_J11: now also FPGA.GPIO_115
- net SIN78_J12: now also FPGA.GPIO_111
- net SIN78_J13: now also FPGA.GPIO_17
- net SIN78_J14: now also FPGA.GPIO_13
- net SIN78_J3: now also FPGA.GPIO_02
- net SIN78_J4: now also FPGA.GPIO_08
- net SIN78_J5: now also FPGA.GPIO_016
- net SIN78_J6: now also FPGA.GPIO_024
- net SIN78_J7: now also FPGA.GPIO_131
- net SIN78_J8: now also FPGA.GPIO_127
- net SIN78_J9: now also FPGA.GPIO_123

Commit message: delete molex keepout footprint, cleaned out backup files
Other:
- moved on the sheet: J10A, J10B, J11A, J11B, J12A, J12B, J13A, J13B, J14A, J14B, J16, J17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

Commit message: Finished power routing and other minor changes
Parts:
- R3, R4: device rcl:R-US_R0402 -> rcl:R-US_R0603
Changed lines of the file:
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@@
 <?xml version="1.0" encoding="utf-8"?>
 <!DOCTYPE eagle SYSTEM "eagle.dtd">
-<eagle version="9.5.2">
+<eagle version="9.6.2">
 <drawing>
 <settings>
@@
 <part name="J19" library="molex" deviceset="436500215" device=""/>
 <part name="R2" library="rcl" library_urn="urn:adsk.eagle:library:334" deviceset="R-US_" device="R0603" package3d_urn="urn:adsk.eagle:package:23555/3" value="165 Ω"/>
-<part name="R3" library="rcl" library_urn="urn:adsk.eagle:library:334" deviceset="R-US_" device="R0402" package3d_urn="urn:adsk.eagle:package:23547/3" value="19.1k Ω"/>
+<part name="R3" library="rcl" library_urn="urn:adsk.eagle:library:334" deviceset="R-US_" device="R0603" package3d_urn="urn:adsk.eagle:package:23555/3" value="19.1k Ω"/>
 <part name="J15" library="molex" deviceset="430450612" device=""/>
 <part name="J18" library="molex" deviceset="436500215" device=""/>
 <part name="J17" library="molex" deviceset="430450612" device=""/>
 <part name="R1" library="rcl" library_urn="urn:adsk.eagle:library:334" deviceset="R-US_" device="R0603" package3d_urn="urn:adsk.eagle:package:23555/3" value="165 Ω"/>
-<part name="R4" library="rcl" library_urn="urn:adsk.eagle:library:334" deviceset="R-US_" device="R0402" package3d_urn="urn:adsk.eagle:package:23547/3" value="19.1k Ω"/>
+<part name="R4" library="rcl" library_urn="urn:adsk.eagle:library:334" deviceset="R-US_" device="R0603" package3d_urn="urn:adsk.eagle:package:23555/3" value="19.1k Ω"/>
 <part name="J16" library="molex" deviceset="430450612" device=""/>
 <part name="C4" library="GTOR - Passive Components" deviceset="CAP_THT" device="E2-5" package3d_urn="urn:adsk.eagle:package:23346/2" value="100u"/>

Commit message: Cleaned schematics, added pdfs
Other:
- note added: "Encoder"
- note added: "FPGA"
- note added: "HDMI"
- note added: "LED Matrix Connections"
- note added: "Logic Buffers"
- note added: "Power"
- note added: "Raspberry Pi"
- note added: "Slip Ring"

Commit message: Fixes to controls board
Parts:
- added C16, C17, C18, C19, C20, C21, C22, C23, C24, C25, C26, C27: 100u, GTOR - Passive Components:CAP_THTE2-5
- added C28, C30, C32: 0.1u, GTOR - Passive Components:CAP_SMDC0603
- added C29, C31, C33: 4.7u, GTOR - Passive Components:CAP_SMDC0603
Connections:
- net 3V3_LOGIC: now also C16.+, C17.+, C18.+, C19.+, C20.+, C21.+, C22.+, C23.+, C24.+, C25.+, C26.+, C27.+, C28.1, C29.1, C30.1, C31.1, C32.1, C33.1
- net GND: now also C16.-, C17.-, C18.-, C19.-, C20.-, C21.-, C22.-, C23.-, C24.-, C25.-, C26.-, C27.-, C28.2, C29.2, C30.2, C31.2, C32.2, C33.2, U$1.GND@1, U$1.GND@2, U$1.GND@3, U$1.GND@4, U$1.GND@5, U$1.GND@6, U$1.GND@7
Other:
- moved on the sheet: C10, C11, C12, C13, C14, C15, C4, C5, C6, C7, C8, C9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
