File: Controls/SpinningControls_preDan.brd (EAGLE design)
At the start: 209.6 x 107.9 mm, 120 parts, among them IC1 S-19246E33H-V5T2U, IC2 SN74LVC1G34DBVR, IC3 SN74LVC1G34DBVR, IC4 SN74LVC1G34DBVR, IC5 TXS0104EDR, J10 SULLINS_PPPC062LFBN-RCSULLINS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, J11 SULLINS_PPPC062LFBN-RCSULLINS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, J12 SULLINS_PPPC062LFBN-RCSULLINS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, J13 SULLINS_PPPC062LFBN-RCSULLINS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, J14 SULLINS_PPPC062LFBN-RCSULLINS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, J15 430450612, J16 430450612, J17 430450612, J18 436500215, J19 436500215, J2 F32R-1A7H1-11040, J3 SULLINS_PPPC062LFBN-RCSULLINS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, J4 SULLINS_PPPC062LFBN-RCSULLINS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, J5 SULLINS_PPPC062LFBN-RCSULLINS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, J6 SULLINS_PPPC062LFBN-RCSULLINS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, J7 SULLINS_PPPC062LFBN-RCSULLINS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, J8 SULLINS_PPPC062LFBN-RCSULLINS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, J9 SULLINS_PPPC062LFBN-RCSULLINS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

Commit message: dan changes + lib
Parts:
- removed C34, C35: 0.1u, GTOR - Passive Components:C0603
- removed C36: 10p, rcl:C0603
- removed IC5: TXS0104EDR, TXS0104EDR:SOIC127P600X175-14N
- removed R10, R11, R12, R13, R14, R15, R16, R17, R18, R19, R21, R22, R23, R24, R25, R26, R27, R28, R29, R30, R31, R32, R33, R34, R35, R36, R37, R38, R39, R40, R41, R42, R43, R44, R45, R46, R47, R48, R49, R5, R50, R51, R52, R53, R54, R55, R56, R6, R7, R8, R9: (no value), rcl:R0402
- removed R20: (no value), rcl:R0603
Connections:
- removed net ENC_POS_SR: IC5.10, J15.4
- removed net N$15: FPGA.47, R6.2
- removed net N$16: FPGA.49, R7.2
- removed net N$17: FPGA.15, R27.2
- removed net N$18: FPGA.53, R8.2
- removed net N$19: FPGA.55, R9.2
- removed net N$2: FPGA.45, R5.2
- removed net N$20: FPGA.57, R10.2
- removed net N$21: FPGA.59, R11.2
- removed net N$22: FPGA.61, R12.2
- removed net N$23: FPGA.63, R13.2
- removed net N$24: FPGA.65, R14.2
- removed net N$25: FPGA.67, R15.2
- removed net N$26: FPGA.17, R28.2
- removed net N$27: FPGA.71, R16.2
- removed net N$28: FPGA.73, R17.2
- removed net N$29: FPGA.75, R18.2
- removed net N$30: FPGA.77, R19.2
- removed net N$31: FPGA.19, R29.2
- removed net N$32: FPGA.21, R30.2
- removed net N$33: FPGA.23, R31.2
- removed net N$34: FPGA.25, R32.2
- removed net N$35: FPGA.27, R33.2
- removed net N$36: FPGA.31, R34.2
- removed net N$37: FPGA.33, R35.2
- removed net N$38: FPGA.35, R36.2
- removed net N$39: FPGA.37, R37.2
- removed net N$40: FPGA.39, R38.2
- removed net N$41: FPGA.14, R44.1
- removed net N$42: FPGA.16, R45.1
- removed net N$43: FPGA.18, R46.1
- removed net N$44: FPGA.20, R47.1
- removed net N$45: FPGA.22, R48.1
- removed net N$46: FPGA.24, R49.1
- removed net N$47: FPGA.26, R50.1
- removed net N$48: FPGA.28, R51.1
- removed net N$49: FPGA.32, R52.1
- removed net N$5: FPGA.79, R21.2
- removed net N$50: FPGA.34, R53.1
- removed net N$51: FPGA.36, R54.1
- removed net N$52: FPGA.38, R55.1
- removed net N$53: FPGA.40, R56.1
- removed net N$54: FPGA.2, R39.1
- removed net N$8: FPGA.7, R24.2
- removed net PI_RX_SR: C36.1, IC5.11, J15.5
- removed net PI_TX_SR: IC5.12, J15.6
- net 3V3_LOGIC: no longer C34.1, IC5.1, IC5.8, R20.2
- net 5V: no longer C35.1, IC5.14
- net ENC_POS: now also J15.4; no longer IC5.5
- net GND: no longer C34.2, C35.2, C36.2, IC5.7, R20.1
- net GSCLK_FPGA: now also FPGA.79; no longer R21.1
- net LAT_FPGA: now also FPGA.39; no longer R38.1
- net N$10: now also FPGA.30; no longer FPGA.4, R40.1
- net N$11: now also FPGA.51; no longer FPGA.6, R41.1
- net N$12: now also FPGA.69; no longer FPGA.8, R42.1
- net N$13: now also FPGA.52; no longer FPGA.10, R43.1
- net N$14: now also FPGA.70; no longer FPGA.13, R26.2
- net N$3: now also FPGA.11; no longer FPGA.50, R22.1
- net N$7: now also FPGA.12; no longer FPGA.5, R23.2
- net N$9: now also FPGA.29; no longer FPGA.9, R25.2
- net PI_RX: now also J15.5; no longer IC5.4
- net PI_TX: now also J15.6; no longer IC5.3
- net SCLK_FPGA: now also FPGA.40; no longer R56.2
- net SIN12_J10: now also FPGA.21; no longer R30.1
- net SIN12_J11: now also FPGA.17; no longer R28.1
- net SIN12_J12: now also FPGA.13; no longer R26.1
- net SIN12_J13: now also FPGA.7; no longer R24.1
- net SIN12_J14: now also FPGA.2; no longer R39.2
- net SIN12_J3: now also FPGA.50; no longer R22.2
- net SIN12_J4: now also FPGA.59; no longer R11.1
- net SIN12_J5: now also FPGA.67; no longer R15.1
- net SIN12_J6: now also FPGA.77; no longer R19.1
- net SIN12_J7: now also FPGA.35; no longer R36.1
- net SIN12_J8: now also FPGA.31; no longer R34.1
- net SIN12_J9: now also FPGA.25; no longer R32.1
- net SIN34_J10: now also FPGA.22; no longer R48.2
- net SIN34_J11: now also FPGA.18; no longer R46.2
- net SIN34_J12: now also FPGA.14; no longer R44.2
- net SIN34_J13: now also FPGA.8; no longer R42.2
- net SIN34_J14: now also FPGA.4; no longer R40.2
- net SIN34_J3: now also FPGA.49; no longer R7.1
- net SIN34_J4: now also FPGA.57; no longer R10.1
- net SIN34_J5: now also FPGA.65; no longer R14.1
- net SIN34_J6: now also FPGA.75; no longer R18.1
- net SIN34_J7: now also FPGA.36; no longer R54.2
- net SIN34_J8: now also FPGA.32; no longer R52.2
- net SIN34_J9: now also FPGA.26; no longer R50.2
- net SIN56_J10: now also FPGA.23; no longer R31.1
- net SIN56_J11: now also FPGA.19; no longer R29.1
- net SIN56_J12: now also FPGA.15; no longer R27.1
- net SIN56_J13: now also FPGA.9; no longer R25.1
- net SIN56_J14: now also FPGA.5; no longer R23.1
- net SIN56_J3: now also FPGA.47; no longer R6.1
- net SIN56_J4: now also FPGA.55; no longer R9.1
- net SIN56_J5: now also FPGA.63; no longer R13.1
- net SIN56_J6: now also FPGA.73; no longer R17.1
- net SIN56_J7: now also FPGA.37; no longer R37.1
- net SIN56_J8: now also FPGA.33; no longer R35.1
- net SIN56_J9: now also FPGA.27; no longer R33.1
- net SIN78_J10: now also FPGA.24; no longer R49.2
- net SIN78_J11: now also FPGA.20; no longer R47.2
- net SIN78_J12: now also FPGA.16; no longer R45.2
- net SIN78_J13: now also FPGA.10; no longer R43.2
- net SIN78_J14: now also FPGA.6; no longer R41.2
- net SIN78_J3: now also FPGA.45; no longer R5.1
- net SIN78_J4: now also FPGA.53; no longer R8.1
- net SIN78_J5: now also FPGA.61; no longer R12.1
- net SIN78_J6: now also FPGA.71; no longer R16.1
- net SIN78_J7: now also FPGA.38; no longer R55.2
- net SIN78_J8: now also FPGA.34; no longer R53.2
- net SIN78_J9: now also FPGA.28; no longer R51.2
Routing:
- net SIN12_J14: track 15.5 -> 69.5 mm
- net GSCLK_FPGA: track 35.8 -> 80.3 mm
- net SIN12_J6: track 68.8 -> 111.0 mm
- net SIN34_J6: track 67.4 -> 107.3 mm
- net SIN56_J6: track 72.3 -> 109.8 mm
- net SIN78_J6: track 71.0 -> 106.2 mm
- net SIN12_J5: track 74.6 -> 107.5 mm
- net SIN34_J5: track 73.1 -> 103.7 mm
- net SIN56_J5: track 77.7 -> 105.9 mm
- net SIN78_J5: track 76.3 -> 102.2 mm
- net SIN12_J4: track 85.7 -> 109.2 mm
- net SIN34_J4: track 84.5 -> 105.7 mm
- net SIN56_J4: track 89.2 -> 108.0 mm
- net SIN78_J4: track 87.7 -> 104.2 mm
- net SIN34_J3: track 108.9 -> 120.8 mm
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