File: Controls/SpinningControls_toOptimize.brd (EAGLE design)
At the start: 209.6 x 107.9 mm, 120 parts, among them IC1 S-19246E33H-V5T2U, IC2 SN74LVC1G34DBVR, IC3 SN74LVC1G34DBVR, IC4 SN74LVC1G34DBVR, IC5 TXS0104EDR, J10 SULLINS_PPPC062LFBN-RCSULLINS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, J11 SULLINS_PPPC062LFBN-RCSULLINS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, J12 SULLINS_PPPC062LFBN-RCSULLINS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, J13 SULLINS_PPPC062LFBN-RCSULLINS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, J14 SULLINS_PPPC062LFBN-RCSULLINS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

Commit message: dan tings, 50ohm FPGA inline, 3v3 to 5 logic for SR
Parts:
- moved R44 190.2 mm to (-53.3, 34.3)
- moved R45 190.2 mm to (-49.5, 34.3)
- moved R46 190.2 mm to (-45.7, 34.3)
- moved R47 190.2 mm to (-41.9, 34.3)
- moved R48 190.2 mm to (-38.1, 34.3)
- moved R49 190.2 mm to (-34.3, 34.3)
- moved R50 190.2 mm to (-30.5, 34.3)
- moved R51 190.2 mm to (-26.7, 34.3)
- moved R52 190.2 mm to (-22.9, 34.3)
- moved R53 190.2 mm to (-19.1, 34.3)
- moved R54 190.2 mm to (-15.2, 34.3)
- moved R55 190.2 mm to (-11.4, 34.3)
- moved R56 190.2 mm to (-7.62, 34.3)
- moved R42 128.0 mm to (-61.0, 34.3), turned to 90 degrees
- moved R43 118.0 mm to (-57.1, 34.3), turned to 90 degrees
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Connections:
- net N$10: now also FPGA.4; no longer FPGA.9
- net N$11: now also FPGA.6; no longer FPGA.7
- net N$12: now also FPGA.8; no longer FPGA.5
- net N$13: now also FPGA.10; no longer FPGA.2
- net N$54: now also FPGA.2; no longer FPGA.10
- net N$7: now also FPGA.5; no longer FPGA.8
- net N$8: now also FPGA.7; no longer FPGA.6
- net N$9: now also FPGA.9; no longer FPGA.4
Routing:
- net SIN12_J14: track 70.6 -> 15.5 mm
- net GSCLK: track 411.5 -> 399.5 mm
- net SCLK: track 366.2 -> 354.5 mm
- net LAT: track 388.5 -> 378.8 mm
- net SIN34_J14: track 73.3 -> 66.1 mm
- net SIN78_J14: track 71.0 -> 65.1 mm
- net N$54: track 5.59 -> 0.00 mm
- net N$8: track 5.48 -> 0.00 mm
- net N$7: track 5.29 -> 0.00 mm
- net N$9: track 5.21 -> 0.00 mm
- net SIN56_J13: track 55.7 -> 60.8 mm
- net SIN12_J13: track 56.7 -> 60.8 mm
- net GND: track 60.8 -> 57.0 mm
- net N$11: track 2.54 -> 0.00 mm
- net N$12: track 2.33 -> 0.00 mm
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