File: LEDSubMatrix_rev2/LEDSubMatrixHighDensity/Backup/LEDSubMatrixHighDensity_template.sch (EAGLE design)
At the start: 138 parts, among them IC1 TLC5955DCAR, IC2 TLC5955DCAR, IC3 TLC5955DCAR, IC4 TLC5955DCAR, IC5 TLC5955DCAR, IC6 TLC5955DCAR, IC7 TLC5955DCAR, IC8 TLC5955DCAR

Commit message: Updated pinouts to align with control board
Parts:
- removed C9: 20uF, rcl:C-EUC0805
- added C1B, C2B, C3B, C4B, C5B, C6B, C7B, C8B: 10uF, rcl:C-EUC0402
- C1, C2, C3, C4, C5, C6, C7, C8: value 20uF -> .1uF; device rcl:C-EUC0603 -> rcl:C-EUC0402
Connections:
- new net 3V3_LOGIC: C1.1, C1B.1, C2.1, C2B.1, C3.1, C3B.1, C4.1, C4B.1, C5.1, C5B.1, C6.1, C6B.1, C7.1, C7B.1, C8.1, C8B.1, IC1.VCC, IC2.VCC, IC3.VCC, IC4.VCC, IC5.VCC, IC6.VCC, IC7.VCC, IC8.VCC, SV1.9
- net 3V3: no longer C1.1, C2.1, C3.1, C4.1, C5.1, C6.1, C7.1, C8.1, C9.1, IC1.VCC, IC2.VCC, IC3.VCC, IC4.VCC, IC5.VCC, IC6.VCC, IC7.VCC, IC8.VCC
- net GND: now also C1B.2, C2B.2, C3B.2, C4B.2, C5B.2, C6B.2, C7B.2, C8B.2; no longer C9.2, SV1.9
Other:
- moved on the sheet: C1, C2, C3, C4, C5, C6, C7, C8
