File: LEDSubMatrix_rev2/LEDSubMatrixHighDensity/Backup/LEDSubMatrixHighDensity_test.brd (EAGLE design)
At the start: 160 x 100 mm, 138 parts, among them IC1 TLC5955DCAR, IC2 TLC5955DCAR, IC3 TLC5955DCAR, IC4 TLC5955DCAR, IC5 TLC5955DCAR, IC6 TLC5955DCAR, IC7 TLC5955DCAR, IC8 TLC5955DCAR

Commit message: Updated pinouts to align with control board
Parts:
- removed C9: 20uF, rcl:C0805
- added C1B, C2B, C3B, C4B, C5B, C6B, C7B, C8B: 10uF, rcl:C0402
- C1, C2, C3, C4, C5, C6, C7, C8: value 20uF -> .1uF; device rcl:C0603 -> rcl:C0402
- SV1: device con-lstb:MA06-2 -> VoxelEagleLib:MA06-2
- moved C8 256.8 mm to (13.8, -138.4), flipped to the bottom, turned to 270 degrees
- moved C6 251.2 mm to (13.8, -104.6), flipped to the bottom, turned to 270 degrees
- moved C7 239.2 mm to (13.8, -121.5), flipped to the bottom, turned to 270 degrees
- moved C5 233.5 mm to (13.8, -87.6), flipped to the bottom, turned to 270 degrees
- moved C4 215.8 mm to (13.8, -70.7), flipped to the bottom, turned to 270 degrees
- moved C3 198.2 mm to (13.8, -53.8), flipped to the bottom, turned to 270 degrees
- moved C2 180.7 mm to (13.8, -36.8), flipped to the bottom, turned to 270 degrees
- moved SV1 168.3 mm to (8.63, -142.0)
- moved C1 163.4 mm to (13.8, -19.9), flipped to the bottom, turned to 270 degrees
- moved LED117 100.5 mm to (2.12, -131.9)
- moved LED118 100.3 mm to (6.35, -131.9)
- moved LED119 100.2 mm to (10.6, -131.9)
- moved LED120 100.2 mm to (14.8, -131.9)
- moved LED116 96.1 mm to (14.8, -127.7)
- moved LED115 96.0 mm to (10.6, -127.7)
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Connections:
- removed net N$1: SV1.1
- removed net N$364: IC8.41
- removed net N$365: IC8.40
- removed net N$366: IC8.39
- removed net N$367: IC8.38
- removed net N$368: IC8.37
- removed net N$369: IC8.36
- removed net N$370: IC8.35
- removed net N$371: IC8.34
- removed net N$372: IC8.33
- removed net N$373: IC8.32
- removed net N$374: IC8.31
- removed net N$375: IC8.30
- net 3V3: now also C1B.1, C2B.1, C3B.1, C4B.1, C5B.1, C6B.1, C7B.1, C8B.1, SV1.6, SV1.8; no longer C9.1, SV1.10, SV1.9
- net GND: now also C1B.2, C2B.2, C3B.2, C4B.2, C5B.2, C6B.2, C7B.2, C8B.2, SV1.10, SV1.9; no longer C9.2, SV1.11
- net GSCLK: now also SV1.11; no longer SV1.6
- net LAT: now also SV1.5; no longer SV1.8
- net N$LEDB109: now also IC7.4; no longer IC7.6
- net N$LEDB110: now also IC7.7; no longer IC7.9
- net N$LEDB115: now also IC8.32
- net N$LEDB116: now also IC8.35
- net N$LEDB119: now also IC8.38
- net N$LEDB120: now also IC8.41
- net N$LEDB13: now also IC1.4; no longer IC1.6
- net N$LEDB14: now also IC1.7; no longer IC1.9
- net N$LEDB29: now also IC2.4; no longer IC2.6
- net N$LEDB30: now also IC2.7; no longer IC2.9
- net N$LEDB45: now also IC3.4; no longer IC3.6
- net N$LEDB46: now also IC3.7; no longer IC3.9
- net N$LEDB61: now also IC4.4; no longer IC4.6
- net N$LEDB62: now also IC4.7; no longer IC4.9
- net N$LEDB77: now also IC5.4; no longer IC5.6
- net N$LEDB78: now also IC5.7; no longer IC5.9
- net N$LEDB93: now also IC6.4; no longer IC6.6
- net N$LEDB94: now also IC6.7; no longer IC6.9
- net N$LEDG109: now also IC7.6; no longer IC7.4
- net N$LEDG110: now also IC7.9; no longer IC7.7
- net N$LEDG115: now also IC8.30
- net N$LEDG116: now also IC8.33
- net N$LEDG119: now also IC8.36
- net N$LEDG120: now also IC8.39
- net N$LEDG13: now also IC1.6; no longer IC1.4
- net N$LEDG14: now also IC1.9; no longer IC1.7
- net N$LEDG29: now also IC2.6; no longer IC2.4
- net N$LEDG30: now also IC2.9; no longer IC2.7
- net N$LEDG45: now also IC3.6; no longer IC3.4
- net N$LEDG46: now also IC3.9; no longer IC3.7
- net N$LEDG61: now also IC4.6; no longer IC4.4
- net N$LEDG62: now also IC4.9; no longer IC4.7
- net N$LEDG77: now also IC5.6; no longer IC5.4
- net N$LEDG78: now also IC5.9; no longer IC5.7
- net N$LEDG93: now also IC6.6; no longer IC6.4
- net N$LEDG94: now also IC6.9; no longer IC6.7
- net N$LEDR115: now also IC8.31
- net N$LEDR116: now also IC8.34
- net N$LEDR119: now also IC8.37
- net N$LEDR120: now also IC8.40
- net SCLK: now also SV1.1; no longer SV1.7
- net SIN_7,8: now also SV1.7; no longer SV1.5
Routing:
- net 3V3: track 0.00 -> 25.8 mm, vias 0 -> 14
- net GSCLK: track 0.00 -> 19.5 mm, vias 0 -> 1
- net SCLK: track 0.00 -> 19.3 mm, vias 0 -> 1
- net LAT: track 0.00 -> 18.3 mm, vias 0 -> 1
- net N$LEDB32: track 0.00 -> 11.6 mm, vias 0 -> 1
- net N$LEDB16: track 0.00 -> 11.6 mm, vias 0 -> 1
- net N$LEDR32: track 0.00 -> 10.1 mm, vias 0 -> 1
- net N$LEDR16: track 0.00 -> 10.1 mm, vias 0 -> 1
- net N$LEDG16: track 0.00 -> 8.57 mm, vias 0 -> 1
- net N$LEDG32: track 0.00 -> 8.57 mm, vias 0 -> 1
- net N$LEDB6: track 0.00 -> 8.49 mm, vias 0 -> 1
- net N$LEDB22: track 0.00 -> 8.49 mm, vias 0 -> 1
- net N$LEDR30: track 0.00 -> 8.25 mm, vias 0 -> 1
- net N$LEDR14: track 0.00 -> 8.25 mm, vias 0 -> 1
- net N$LEDG11: track 0.00 -> 8.10 mm, vias 0 -> 1
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- added copper zone on layer 15, net 3V3
- added copper zone on layer 2, net GND
Other:
- board size 160 x 100 mm -> 16.9 x 146 mm
