File: LEDSubMatrix_rev2/LEDSubMatrixHighDensity/Backup/LEDSubMatrixHighDensity_test.sch (EAGLE design)
At the start: 138 parts, among them IC1 TLC5955DCAR, IC2 TLC5955DCAR, IC3 TLC5955DCAR, IC4 TLC5955DCAR, IC5 TLC5955DCAR, IC6 TLC5955DCAR, IC7 TLC5955DCAR, IC8 TLC5955DCAR

Commit message: Updated pinouts to align with control board
Parts:
- removed C9: 20uF, rcl:C-EUC0805
- added C1B, C2B, C3B, C4B, C5B, C6B, C7B, C8B: 10uF, rcl:C-EUC0402
- C1, C2, C3, C4, C5, C6, C7, C8: value 20uF -> .1uF; device rcl:C-EUC0603 -> rcl:C-EUC0402
- SV1: device con-lstb:MA06-2 -> VoxelEagleLib:MA06-2
Connections:
- removed net N$1: SV1.1
- removed net N$364: IC8.OUTB14
- removed net N$365: IC8.OUTR14
- removed net N$366: IC8.OUTG14
- removed net N$367: IC8.OUTB10
- removed net N$368: IC8.OUTR10
- removed net N$369: IC8.OUTG10
- removed net N$370: IC8.OUTB15
- removed net N$371: IC8.OUTR15
- removed net N$372: IC8.OUTG15
- removed net N$373: IC8.OUTB11
- removed net N$374: IC8.OUTR11
- removed net N$375: IC8.OUTG11
- net 3V3: now also C1B.1, C2B.1, C3B.1, C4B.1, C5B.1, C6B.1, C7B.1, C8B.1, SV1.6, SV1.8; no longer C9.1, SV1.10, SV1.9
- net GND: now also C1B.2, C2B.2, C3B.2, C4B.2, C5B.2, C6B.2, C7B.2, C8B.2, SV1.10, SV1.9; no longer C9.2, SV1.11
- net GSCLK: now also SV1.11; no longer SV1.6
- net LAT: now also SV1.5; no longer SV1.8
- net N$LEDB109: now also IC7.OUTB4; no longer IC7.OUTG4
- net N$LEDB110: now also IC7.OUTB0; no longer IC7.OUTG0
- net N$LEDB115: now also IC8.OUTB11
- net N$LEDB116: now also IC8.OUTB15
- net N$LEDB119: now also IC8.OUTB10
- net N$LEDB120: now also IC8.OUTB14
- net N$LEDB13: now also IC1.OUTB4; no longer IC1.OUTG4
- net N$LEDB14: now also IC1.OUTB0; no longer IC1.OUTG0
- net N$LEDB29: now also IC2.OUTB4; no longer IC2.OUTG4
- net N$LEDB30: now also IC2.OUTB0; no longer IC2.OUTG0
- net N$LEDB45: now also IC3.OUTB4; no longer IC3.OUTG4
- net N$LEDB46: now also IC3.OUTB0; no longer IC3.OUTG0
- net N$LEDB61: now also IC4.OUTB4; no longer IC4.OUTG4
- net N$LEDB62: now also IC4.OUTB0; no longer IC4.OUTG0
- net N$LEDB77: now also IC5.OUTB4; no longer IC5.OUTG4
- net N$LEDB78: now also IC5.OUTB0; no longer IC5.OUTG0
- net N$LEDB93: now also IC6.OUTB4; no longer IC6.OUTG4
- net N$LEDB94: now also IC6.OUTB0; no longer IC6.OUTG0
- net N$LEDG109: now also IC7.OUTG4; no longer IC7.OUTB4
- net N$LEDG110: now also IC7.OUTG0; no longer IC7.OUTB0
- net N$LEDG115: now also IC8.OUTG11
- net N$LEDG116: now also IC8.OUTG15
- net N$LEDG119: now also IC8.OUTG10
- net N$LEDG120: now also IC8.OUTG14
- net N$LEDG13: now also IC1.OUTG4; no longer IC1.OUTB4
- net N$LEDG14: now also IC1.OUTG0; no longer IC1.OUTB0
- net N$LEDG29: now also IC2.OUTG4; no longer IC2.OUTB4
- net N$LEDG30: now also IC2.OUTG0; no longer IC2.OUTB0
- net N$LEDG45: now also IC3.OUTG4; no longer IC3.OUTB4
- net N$LEDG46: now also IC3.OUTG0; no longer IC3.OUTB0
- net N$LEDG61: now also IC4.OUTG4; no longer IC4.OUTB4
- net N$LEDG62: now also IC4.OUTG0; no longer IC4.OUTB0
- net N$LEDG77: now also IC5.OUTG4; no longer IC5.OUTB4
- net N$LEDG78: now also IC5.OUTG0; no longer IC5.OUTB0
- net N$LEDG93: now also IC6.OUTG4; no longer IC6.OUTB4
- net N$LEDG94: now also IC6.OUTG0; no longer IC6.OUTB0
- net N$LEDR115: now also IC8.OUTR11
- net N$LEDR116: now also IC8.OUTR15
- net N$LEDR119: now also IC8.OUTR10
- net N$LEDR120: now also IC8.OUTR14
- net SCLK: now also SV1.1; no longer SV1.7
- net SIN_7,8: now also SV1.7; no longer SV1.5
Other:
- moved on the sheet: C1, C2, C3, C4, C5, C6, C7, C8, IC1, IC2, IC3, IC4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
