File: Controls/rev1_backup/SpinningControls.brd (EAGLE design)
At the start: 209.6 x 107.9 mm, 120 parts, among them IC1 S-19246E33H-V5T2U, IC2 SN74LVC1G34DBVR, IC3 SN74LVC1G34DBVR, IC4 SN74LVC1G34DBVR, IC5 TXS0104EDR, J10 SULLINS_PPPC062LFBN-RCSULLINS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, J11 SULLINS_PPPC062LFBN-RCSULLINS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, J12 SULLINS_PPPC062LFBN-RCSULLINS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, J13 SULLINS_PPPC062LFBN-RCSULLINS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, J14 SULLINS_PPPC062LFBN-RCSULLINS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

Commit message: silkscreen update
Other:
- board text removed: "24V"
- board text removed: "5V (FPGA)"
- board text removed: "ENCODER"
- board text removed: "ENCODER0"
- board text removed: "JP0"
- board text removed: "JP1 GPIO0"
- board text removed: "JP2 GPIO1"
- board text removed: "SIN"
